File: MotoComm.sch (KiCad schematic (older format))
At the start: 18 parts

Commit message: first draft with pcb
Parts:
- removed J?: Button_Voltage_Selector, symbol Conn_02x02_Counter_Clockwise
- added C1: 0.1µ, Capacitors_SMD:C_0805_HandSoldering, symbol C
- added C2, C3, C4, C5, C6: 1µ, Capacitors_SMD:C_0805_HandSoldering, symbol C
- added J2: Audio-Jack-3, Connectors:Stereo_Jack_3.5mm_Switch_Ledino_KB3SPRS, symbol Audio-Jack-3
- added J3: Conn_01x03, Pin_Headers:Pin_Header_Straight_1x03_Pitch2.54mm, symbol Conn_01x03
- added J4: Conn_02x01, Connectors_JST:JST_ACH_BM02B-ACHSS_02x1.20mm_Angled, symbol Conn_02x01
- added J5: USB_OTG, Connectors:USB_Micro-B, symbol USB_OTG
- added R10, R11, R4, R5, R6, R7, R8, R9: 100k, Resistors_SMD:R_0805_HandSoldering, symbol R
- added U1: LM358, Housings_SSOP:TSSOP-8_3x3mm_Pitch0.65mm, symbol LM358
- added U3: LT6656**S6, TO_SOT_Packages_SMD:TSOT-23-8_HandSoldering, symbol LT6656**S6
- D1, D3, D5: renamed from D?; footprint (none) -> LEDs:LED_1206_HandSoldering
- D2, D4: renamed from D?; footprint (none) -> Diodes_SMD:D_1206
- J1: renamed from J?; footprint (none) -> Pin_Headers:Pin_Header_Straight_2x05_Pitch2.54mm
- R1, R12, R2, R3: renamed from R?; footprint (none) -> Resistors_SMD:R_0805_HandSoldering
- SW1, SW2, SW3, SW4, SW5, SW6: renamed from SW?; footprint (none) -> Buttons_Switches_THT:SW_TH_Tactile_Omron_B3F-10xx
- U2: renamed from U?; footprint (none) -> modules:F-3188_CSR8645_no_silk_under_antena
Connections:
- net labels added: SPKR_L_N, SPKR_L_P, SPKR_R_N, SPKR_R_P, SPRK_L_OUT, SPRK_R_OUT, USB_N, USB_P, VBUS, VREF
- wire segments 69 -> 136
- no-connect marks 0 -> 14

Commit message: minor update
Parts:
- added C? (x2): CP, symbol CP
Connections:
- wire segments 136 -> 143
Other:
- moved on the sheet: C1, C2, C3, C4, C5, C6, J2, J5, R10, R11, R4, R5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
